File: RS1_PCB_addon.kicad_sch (KiCad schematic)
At the start: 35 parts, among them J1 Conn_01x02, J10 Conn_01x02, J2 SJ-3523-SMT-TR, J3 Conn_01x10_Socket, J4 Conn_01x11, J5 Conn_01x05, J6 Conn_01x02, J7 Conn_01x02, J8 Conn_01x02, J9 Conn_01x02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

Commit message: change edgecut
Parts:
- removed J4: Conn_01x11, Connector_PinSocket_2.54mm:PinSocket_1x11_P2.54mm_Vertical, symbol Connector_Generic:Conn_01x11
- removed J6, J7, J8: Conn_01x02, Connector_PinHeader_2.54mm:PinHeader_1x02_P2.54mm_Vertical, symbol Connector_Generic:Conn_01x02
- J5: footprint Connector_PinHeader_2.54mm:PinHeader_1x05_P2.54mm_Vertical_SMD_Pin1Right -> Connector_PinHeader_2.54mm:PinHeader_1x05_P2.54mm_Vertical
Other:
- note removed: "Connector Addon"
