File: RS1_PCB_addon.kicad_pcb (KiCad board)
At the start: 2 copper layers, 45.6 x 35.6 mm, 31 parts, among them J1 Conn_01x02, J10 Conn_01x02, J2 SJ-3523-SMT-TR, J3 Conn_01x10_Socket, J5 Conn_01x05, J9 Conn_01x02, P2 S2B-PH-SM4-TB, U1 TPS2113ADRBR, U11 LTV-217-B-G, U12 LTV-217-B-G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

Commit message: change edgecut
Parts:
- C1, C2, F2, R14, R15, R16, R17, R18, R2, R5, U1, U3, U4: moved to B.Cu
- J5: footprint Connector_PinHeader_2.54mm:PinHeader_1x05_P2.54mm_Vertical_SMD_Pin1Right -> Connector_PinHeader_2.54mm:PinHeader_1x05_P2.54mm_Vertical; moved to F.Cu
- moved P2 98.0 mm to (128.4, 66.5), turned to 90 degrees
- moved R20 88.1 mm to (124.0, 71.6), turned to 0 degrees
- moved C10 86.4 mm to (127.2, 48.7)
- moved C11 86.1 mm to (127.2, 52.8), turned to 180 degrees
- moved F2 84.3 mm to (120.5, 65.5), turned to 90 degrees
- moved U12 79.7 mm to (121.3, 73.8), turned to 180 degrees
- moved J2 74.5 mm to (109.9, 73.9), turned to 90 degrees
- moved U3 65.1 mm to (104.9, 59.8), turned to -90 degrees
- moved J3 64.6 mm to (93.1, 46.4)
- moved R15 63.4 mm to (107.2, 52.3), turned to -90 degrees
- moved R14 61.8 mm to (106.0, 52.3), turned to -90 degrees
- moved J1 60.9 mm to (114.7, 39.9), turned to 0 degrees
- moved J10 60.9 mm to (124.3, 40.7), turned to 0 degrees
- moved R17 59.0 mm to (102.6, 55.6), turned to 45 degrees
- moved U11 58.5 mm to (101.5, 71.4), turned to -90 degrees
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Routing:
- net /VBAT: track 0.00 -> 55.5 mm, vias 0 -> 2
- net /Op_2: track 0.00 -> 36.7 mm, vias 0 -> 2
- net Net-(J2-Pad1): track 0.00 -> 18.6 mm, vias 0 -> 2
- net /SERVO_PWM: track 0.00 -> 17.5 mm
- net +5V: track 0.00 -> 15.1 mm, vias 0 -> 1
- net GND: track 0.00 -> 13.7 mm, vias 0 -> 4
- net /VSYS: track 0.00 -> 13.0 mm, vias 0 -> 2
- net Net-(J2-Pad2): track 0.00 -> 12.3 mm, vias 0 -> 2
- net /Op_1: track 0.00 -> 12.1 mm
- net /INT_B: track 0.00 -> 11.1 mm, vias 0 -> 1
- net /SDA: track 0.00 -> 10.7 mm
- net /SCL: track 0.00 -> 9.16 mm
- net /STAT_Power_Path: track 0.00 -> 8.50 mm
- net Net-(F2-Pad1): track 0.00 -> 7.98 mm
- net Net-(U4-A0): track 0.00 -> 7.93 mm
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- added copper zone on B.Cu, net GND
- added copper zone on F.Cu, net GND
Other:
- board size 45.6 x 35.6 mm -> 47.5 x 39.5 mm

Commit message: change layout
Parts:
- C10, C11, C8, R4, R7, R8, U5: moved to B.Cu
- moved R18 32.5 mm to (135.2, 55.6), turned to 0 degrees
- moved U3 29.5 mm to (133.7, 53.3), turned to 180 degrees
- moved R15 25.2 mm to (132.0, 57.0), turned to 180 degrees
- moved R14 25.0 mm to (130.7, 56.0), turned to 180 degrees
- moved U4 23.3 mm to (123.8, 54.4)
- moved R17 22.0 mm to (124.2, 59.8), turned to -135 degrees
- moved R16 19.5 mm to (121.8, 59.4), turned to -90 degrees
- moved R8 11.1 mm to (121.2, 42.0)
- moved R7 10.4 mm to (119.1, 44.8)
- moved C8 10.1 mm to (119.1, 39.5)
- moved U5 9.27 mm to (118.5, 42.6)
- moved R4 6.75 mm to (116.8, 46.0), turned to 180 degrees
- moved C11 3.56 mm to (130.4, 51.1), turned to -135 degrees
- moved C10 2.23 mm to (128.7, 50.4), turned to 45 degrees
- moved P2 1.92 mm to (127.6, 68.2)
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Routing:
- net +3.3V: track 0.00 -> 49.8 mm, vias 0 -> 4
- net /SDA: track 10.7 -> 48.2 mm, vias 0 -> 3
- net /SCL: track 9.16 -> 44.8 mm, vias 0 -> 3
- net /Op_2: track 36.7 -> 18.7 mm, vias 2 -> 1
- net /Op_1: track 12.1 -> 27.2 mm, vias 0 -> 2
- net GND: track 13.7 -> 24.4 mm, vias 4 -> 9
- net /STAT_Power_Path: track 8.50 -> 1.11 mm
- net Net-(U4-A0): track 7.93 -> 14.0 mm
- net /VBAT: track 55.5 -> 51.4 mm, vias 2 -> 1
- net /INT_B: track 11.1 -> 15.1 mm
- net Net-(F2-Pad1): track 7.98 -> 9.29 mm, vias 0 -> 2
- net Net-(U4-~{RESET}): track 1.36 -> 2.19 mm

Commit message: change pin position
Parts:
- moved J5 11.0 mm to (110.9, 50.0), turned to 0 degrees
- moved J9 3.26 mm to (95.6, 39.7)
- moved J10 1.18 mm to (123.6, 39.8)
- moved R4 1.11 mm to (116.7, 44.9)
- moved J1 0.90 mm to (113.8, 39.8)
- moved C1 0.70 mm to (109.4, 43.9)
- moved C2 0.51 mm to (110.5, 39.7)
- moved J3 0.30 mm to (93.1, 46.1)
Routing:
- net /MOSFET_SERVO: track 0.00 -> 59.6 mm, vias 0 -> 1
- net /LIGHT_DETECT: track 0.00 -> 41.7 mm, vias 0 -> 3
- net /LED_Switch: track 0.00 -> 41.3 mm, vias 0 -> 1
- net /SERVO_DETECT: track 0.00 -> 35.6 mm, vias 0 -> 3
- net /VBAT: track 51.4 -> 79.1 mm, vias 1 -> 0
- net /STAT_Power_Path: track 1.11 -> 27.8 mm, vias 0 -> 2
- net /PWM_LED: track 0.00 -> 20.7 mm, vias 0 -> 1
- net /BAT_ALERT: track 0.00 -> 15.8 mm, vias 0 -> 2
- net GND: track 24.4 -> 39.6 mm, vias 9 -> 51
- net /SCL: track 44.8 -> 56.8 mm, vias 3 -> 2
- net /SDA: track 48.2 -> 56.1 mm, vias 3 -> 2
- net /SERVO_PWM: track 17.5 -> 22.4 mm, vias 0 -> 1
- net +5V: track 15.1 -> 19.1 mm
- net /Op_1: track 27.2 -> 28.6 mm
- net /INT_B: track 15.1 -> 14.4 mm
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Other:
- board text added: "0x21"
